File: External Sensor Schematic.brd (EAGLE design)
At the start: 160 x 100 mm, 13 parts, among them U1 LT1300CN8PBF, U2 LM35CAZ/NOPB, U3 PI_SENSOR_255-5419-ND

Commit message: Completed Board Layout on all 3
Parts:
- added U$1: (no value), ENG_LOGO:ENG_LOGO
- added U$2: (no value), Canada_Flag_Logo:CANADA_FLAG_LOGO
- added U$3, U$4: (no value), SparkFun-Electromechanical:STAND-OFF-TIGHT
- C1, C2, C3: value 100uF -> 100u; device 100uF_Cap:EEU-FR1H101 -> SparkFun-Capacitors:CPOL-RADIAL-1000UF-25V
- D1: value UF4003 -> (none); device diode:DO41-10 -> SparkFun-DiscreteSemi:DIODE-1N4148
- moved C3 235.0 mm to (38.7, 40.0), turned to 90 degrees
- moved C2 207.7 mm to (26.0, 31.1), turned to 90 degrees
- moved D1 180.4 mm to (13.3, 48.3)
- moved L2 180.2 mm to (38.7, 22.9), turned to 90 degrees
- moved C1 160.8 mm to (13.3, 40.0), turned to 90 degrees
- moved U1 136.3 mm to (17.8, 25.4), flipped to the bottom, turned to 270 degrees
- moved BAT2 116.1 mm to (12.7, 64.8), turned to 90 degrees
- moved L1 101.3 mm to (13.3, 22.9), turned to 90 degrees
- moved U3 97.1 mm to (26.0, 46.4)
- moved BAT1 84.3 mm to (39.4, 64.8), turned to 270 degrees
- moved U2 82.6 mm to (27.3, 4.45)
- moved JP2 75.1 mm to (47.5, 37.5), turned to 270 degrees
- moved JP1 31.3 mm to (4.32, 37.5), turned to 270 degrees
Connections:
- net 3V3: now also C3.+; no longer C3.P
- net GND: now also C2.-, C3.-; no longer C2.G, C3.G
- net N$1: now also C1.+; no longer C1.P
- net N$7: now also C1.-; no longer C1.G
- net VIN: now also C2.+; no longer C2.P
Routing:
- net VIN: track 0.00 -> 93.0 mm
- net TEMP: track 0.00 -> 75.2 mm
- net PROXIMITY: track 0.00 -> 58.6 mm
- net N$7: track 0.00 -> 52.4 mm
- net N$1: track 0.00 -> 46.8 mm
- added copper zone on layer 1, net 3V3
- added copper zone on layer 1, net GND
- added copper zone on layer 16, net GND
Other:
- board size 160 x 100 mm -> 52 x 80 mm
- board text added: "ECE 490/491 Capstone Group 01"
- board text added: "Sensor Controller"
