File: Vent Schematic.sch (EAGLE design)
At the start: 16 parts, among them U1 LT1300CN8PBF, U2 STP10P6F6

Commit message: Completed Board Layout on all 3
Parts:
- removed LED1: (no value), E-P-008-R1.2:LED5MM
- added JP5: (no value), SparkFun-Connectors:M023.5MM
- C1, C2, C3: value 100uF -> 100u; device 100uF_Cap:100UF-POLAR -> SparkFun-Capacitors:1000UF-25V(PTH)
- D1: value UF4003 -> (none); device diode:UF4003 -> SparkFun-DiscreteSemi:DIODE1N4148
- JP3: value (none) -> DF3A-3P-2DS; device SparkFun-Connectors:M03LOCK_LONGPADS -> 3 Pin H3894-ND:DF3A-3P-2DS
- R1, R2, R3: device SparkFun-Passives:RESISTOR0603-RES -> SparkFun-Passives:RESISTORAXIAL-0.3
Connections:
- net GND: now also JP4.2, JP5.2, R3.2; no longer JP4.1, LED1.C, R3.1
- net N$1: now also JP5.1; no longer LED1.A
- net N$3: now also R2.1, R3.1; no longer R2.2, R3.2
- net VIN: now also JP4.1, R2.2; no longer JP4.2, R2.1
Other:
- moved on the sheet: JP4, R2, R3
